Commit message: minichallenge1

File: urdf/puzzlebot.urdf (robot description, URDF)
Before this commit: robot puzzlebot, 5 links, 4 joints
Links:
- removed link caster
- removed link wheel_l
- removed link wheel_r
- added link caster_link
- added link wheel_l_link
- added link wheel_r_link
- link base_link: geometry 
Joints:
- joint base_link_joint: origin xyz=0 0 0.05 rpy=0 0 0 -> xyz=0 0 0.1 rpy=0 0 0
- joint caster_joint: child caster -> caster_link; origin xyz=-0.095 0 -0.03 rpy=0 0 0 -> xyz=-0.1 0 -0.06 rpy=0 0 0
- joint wheel_l_joint: child wheel_l -> wheel_l_link; origin xyz=0.052 0.095 -0.0025 rpy=0 0 0 -> xyz=0.07 0.1 -0.025 rpy=0 0 0
- joint wheel_r_joint: child wheel_r -> wheel_r_link; origin xyz=0.052 -0.095 -0.0025 rpy=0 0 0 -> xyz=0.07 -0.1 -0.025 rpy=0 0 0

Commit message: minichallenge 2

File: urdf/puzzlebot.urdf (robot description, URDF)
Before this commit: robot puzzlebot, 5 links, 4 joints
Links:
- removed link caster_link
- removed link wheel_l_link
- removed link wheel_r_link
- added link caster; visual mesh filename=package://puzzlebot/meshes/Puzzlebot_Caster_Wheel.stl
- added link wheel_l; visual mesh filename=package://puzzlebot/meshes/Puzzlebot_Wheel.stl
- added link wheel_r; visual mesh filename=package://puzzlebot/meshes/Puzzlebot_Wheel.stl
- link base_link: geometry visual mesh filename=package://puzzlebot/meshes/Puzzlebot_Jetson_Lidar_Edition_B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 scale=1 1 1
Joints:
- joint base_link_joint: origin xyz=0 0 0.1 rpy=0 0 0 -> xyz=0 0 0.05 rpy=0 0 0
- joint caster_joint: child caster_link -> caster; origin xyz=-0.1 0 -0.06 rpy=0 0 0 -> xyz=-0.095 0 -0.03 rpy=0 0 0
- joint wheel_l_joint: child wheel_l_link -> wheel_l; origin xyz=0.07 0.1 -0.025 rpy=0 0 0 -> xyz=0.052 0.095 -0.0025 rpy=0 0 0
- joint wheel_r_joint: child wheel_r_link -> wheel_r; origin xyz=0.07 -0.1 -0.025 rpy=0 0 0 -> xyz=0.052 -0.095 -0.0025 rpy=0 0 0
